File: smartMAC - Lamp Detect/smartMAC - Lamp Detect.kicad_sch (KiCad schematic)
At the start: 21 parts, among them J2 Conn_01x01_Pin

Commit message: Lamp detect circuit is now accurate
Parts:
- added C1: 220n, symbol Device:C
- added C2, C3: 3.6u, symbol Device:C
- added C4: 21u, symbol Device:C_Polarized
- added C8: C, symbol Device:C
- added D1: 0.7V, symbol Device:D
- added D2: 0.6V, symbol Device:D
- added PL12: BAL OUT, symbol Connector:Conn_01x01_Pin
- added PL13: BAL IN, symbol Connector:Conn_01x01_Pin
- added PL14: RELAY, symbol Connector:Conn_01x01_Pin
- added R (x2): 0, symbol Device:R
- added R10: 880, symbol Device:R
- added R4: 270k, symbol Device:R
- added R5: 330, symbol Device:R
- added R7: 10k, symbol Device:R
- added R9: 4.7k, symbol Device:R
- added RL1: G2RL-1A-E, Relay_THT:Relay_SPST_Omron_G2RL-1A-E, symbol Relay:G2RL-1A-E
- added U1: TLP131, Package_SO:MFSOP6-5_4.4x3.6mm_P1.27mm, symbol Isolator:TLP131
- C5: value (none) -> ~
- PL11: renamed from J2; value Conn_01x01_Pin -> LAMP
- R2: value 2.8k -> 4.7k
- R3: value 1.8k -> 2.2k
Connections:
- net GND: now also PL1.4 (Pin_4), U2.12 (VCC-), U2.4, U2.5, U2.6, U2.7, U2.8, U2.9, C4.2, C8.1, R10.1, R4.2, R7.2
- net VDC: now also R1.2, R2.2, R3.1
- net at PL11.1 (Pin_1): now also C1.2, PL12.1 (Pin_1)
- net at U2.10: now also R.2
- net at U2.11: now also R3.2, R10.2, R9.1
- net at U2.13: now also PL1.2 (Pin_2), R2.1, R9.2
- net at PL1.3 (Pin_3): now also D2.2 (A), RL1.A1
- net +12V renamed +24V
- net +24V: now also C8.2, D2.1 (K), RL1.A2
- new net: C2.1, C3.1, D1.2 (A), PL13.1 (Pin_1), RL1.14, U1.3
- new net: PL14.1 (Pin_1), RL1.13
- new net: R.1, R.2, R7.1
- new net: C4.1, R.1, U1.4
- new net: C1.1, C2.2, C3.2, D1.1 (K), R5.2
- new net: R5.1, U1.1
- new net: R1.1, U1.5
- new net: R4.1, U1.6
Other:
- note added: "+24VDC Power Supply"
- note removed: "12VDC Power Supply"
- moved on the sheet: C5, PL1, PL11, R1, R2, R3, U2

Commit message: Add notes to Lamp Detect and Hallsensor schematics
Connections:
- net at R10.2, R3.2, U2.11: now also R9.2; no longer R9.1
- net at PL1.2 (Pin_2), R2.1, U2.13: now also R9.1; no longer R9.2
- no-connect marks 0 -> 3
Other:
- note added: "Lamp Detect"
- note added: "Lamp Relay"
- note added: "VDC = +5VDC"
- company: (none) -> Samtronix
- title: (none) -> smartMAC - Lamp Detect (62006024-A)
- moved on the sheet: C5, D2, PL1, R1, R10, R2, R3, R9
